Commit message: Add xacro namespace

File: chapter7_tutorials/rosbook_arm_description/urdf/deg_to_rad.xacro (robot description, xacro)
@@ -1,3 +1,3 @@
 <robot xmlns:xacro="http://ros.org/wiki/xacro">
-  <property name="deg_to_rad" value="0.01745329251994329577"/>
+  <xacro:property name="deg_to_rad" value="0.01745329251994329577"/>
 </robot>

File: chapter7_tutorials/rosbook_arm_description/urdf/inertia.xacro (robot description, xacro)
@@ -3,16 +3,16 @@
        (width, depth and height).
        See http://en.wikipedia.org/wiki/List_of_moments_of_inertia -->
-  <macro name="cuboid_inertia" params="mass x y z">
+  <xacro:macro name="cuboid_inertia" params="mass x y z">
     <inertia ixx="${1/12 * mass * (y * y + z * z)}" ixy="0.0" ixz="0.0"
              iyy="${1/12 * mass * (x * x + z * z)}" iyz="0.0"
              izz="${1/12 * mass * (x * x + y * y)}"/>
-  </macro>
+  </xacro:macro>
   <!-- Moment of inertia tensor for a solid cylinder of given mass, radius and
        length.
        See http://en.wikipedia.org/wiki/List_of_moments_of_inertia -->
-  <macro name="cylinder_inertia" params="mass radius length">
+  <xacro:macro name="cylinder_inertia" params="mass radius length">
     <inertia ixx="${1/12 * mass * (3 * radius * radius + length * length)}" ixy="0.0" ixz="0.0"
              iyy="${1/12 * mass * (3 * radius * radius + length * length)}" iyz="0.0"
              izz="${1/2  * mass * radius * radius}"/>
-  </macro>
+  </xacro:macro>
 </robot>

File: chapter7_tutorials/rosbook_arm_description/urdf/sensors/xtion_pro_live.urdf.xacro (robot description, xacro)
@@ -14,5 +14,5 @@
     <!-- frames in the center of the camera -->
     <joint name="${name}_joint" type="fixed">
-      <insert_block name="origin"/>
+      <xacro:insert_block name="origin"/>
       <parent link="${parent}_link"/>
       <child link="${name}_link"/>
@@ -35,5 +35,5 @@
     </link>
     <joint name="${name}_optical_joint" type="fixed">
-      <insert_block name="optical_origin"/>
+      <xacro:insert_block name="optical_origin"/>
       <parent link="${name}_link"/>
       <child link="${name}_optical_frame"/>
